File: schematics/RF Duinode V3.sch (EAGLE design)
At the start: 22 parts, among them IC2 ATMEGA328, IC3 MCP9700, Q1 8MHz

Commit message: fixed previous commit
Parts:
- removed G2: CR2450H, JC:CR2450H
- JP6: value EXTPWR -> BATT
Connections:
- net EXTPWR renamed BATT
- removed net COIN: G2.+, SW_PWR.S
- new net EXT_VSUPPLY: JP7.4, SW_PWR.S
- net +3V3: no longer JP7.4
- net GND: no longer G2.-
- net GRN_LED: now also R3.2
- net RED_LED: now also R2.1
Other:
- moved on the sheet: R1
Changed lines of the file:
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@@
 <part name="JP7" library="SparkFun" deviceset="FTDI_BASIC" device="PTH"/>
 <part name="SUPPLY17" library="supply2" deviceset="GND" device=""/>
-<part name="JP6" library="SparkFun" deviceset="M02" device="LOCK" value="EXTPWR"/>
+<part name="JP6" library="SparkFun" deviceset="M02" device="LOCK" value="BATT"/>
 <part name="SUPPLY23" library="supply2" deviceset="GND" device=""/>
 <part name="U$2" library="SparkFun" deviceset="M04X2" device="" value="RADIO"/>
@@
 <part name="+3V7" library="supply1" deviceset="+3V3" device=""/>
 <part name="SUPPLY8" library="supply2" deviceset="GND" device=""/>
-<part name="G2" library="JC" deviceset="CR2450H" device=""/>
-<part name="SUPPLY10" library="supply2" deviceset="GND" device=""/>
 <part name="SW_PWR" library="JC" deviceset="SWITCH-SPDT" device=""/>
 <part name="C4" library="resistor" deviceset="C-EU" device="025-025X050" value="0.1uF"/>
@@
 <part name="+3V4" library="supply1" deviceset="+3V3" device=""/>
 <part name="+3V9" library="supply1" deviceset="+3V3" device=""/>
-<part name="+3V10" library="supply1" deviceset="+3V3" device=""/>
 <part name="LED1" library="led" deviceset="L-115WEGW-CA" device=""/>
 <part name="+3V1" library="supply1" deviceset="+3V3" device=""/>
@@
 <instance part="JP2" gate="G$1" x="-124.46" y="15.24"/>
 <instance part="JP8" gate="G$1" x="-121.92" y="17.78"/>
-<instance part="R1" gate="G$1" x="-96.52" y="83.82" rot="R90"/>
+<instance part="R1" gate="G$1" x="-93.98" y="83.82" rot="R90"/>
 <instance part="SUPPLY13" gate="GND" x="-114.3" y="35.56" rot="R270"/>
 <instance part="JP7" gate="G$1" x="-129.54" y="78.74"/>
@@
 <instance part="+3V5" gate="G$1" x="-127" y="45.72" rot="R90"/>
 <instance part="+3V6" gate="G$1" x="-96.52" y="38.1" rot="R90"/>
-<instance part="+3V3" gate="G$1" x="-96.52" y="93.98"/>
+<instance part="+3V3" gate="G$1" x="-93.98" y="93.98"/>
 <instance part="IC3" gate="G$1" x="53.34" y="76.2"/>
 <instance part="+3V7" gate="G$1" x="27.94" y="81.28"/>
 <instance part="SUPPLY8" gate="GND" x="38.1" y="71.12"/>
-<instance part="G2" gate="G$1" x="109.22" y="109.22"/>
-<instance part="SUPPLY10" gate="GND" x="101.6" y="109.22" rot="R270"/>
 <instance part="SW_PWR" gate="BEF1" x="127" y="106.68" rot="R90"/>
 <instance part="C4" gate="G$1" x="30.48" y="73.66" rot="R90"/>
@@
 <instance part="+3V4" gate="G$1" x="139.7" y="106.68" rot="R270"/>
 <instance part="+3V9" gate="G$1" x="124.46" y="10.16" rot="R270"/>
-<instance part="+3V10" gate="G$1" x="-104.14" y="81.28" rot="R270"/>
 <instance part="LED1" gate="G$1" x="73.66" y="40.64" rot="R90"/>
 <instance part="+3V1" gate="G$1" x="73.66" y="30.48" rot="R180"/>
@@
 <pinref part="S1" gate="1" pin="P"/>
 </segment>
-<segment>
-<pinref part="G2" gate="G$1" pin="-"/>
-<pinref part="SUPPLY10" gate="GND" pin="GND"/>
-</segment>
 </net>
 <net name="DTR" class="0">
@@
 <segment>
 <wire x1="66.04" y1="55.88" x2="66.04" y2="58.42" width="0.1524" layer="91"/>
-<label x="66.04" y="55.88" size="1.778" layer="95" rot="R90"/>
+<label x="66.04" y="58.42" size="1.778" layer="95" rot="R90"/>
+<pinref part="R2" gate="G$1" pin="1"/>
+<junction x="66.04" y="55.88"/>
 </segment>
 </net>
@@
 <segment>
 <wire x1="81.28" y1="55.88" x2="81.28" y2="58.42" width="0.1524" layer="91"/>
-<label x="81.28" y="55.88" size="1.778" layer="95" rot="R90"/>
+<label x="81.28" y="58.42" size="1.778" layer="95" rot="R90"/>
+<pinref part="R3" gate="G$1" pin="2"/>
+<junction x="81.28" y="55.88"/>
 </segment>
 </net>
@@
 <net name="RESET" class="0">
 <segment>
-<wire x1="-91.44" y1="73.66" x2="-96.52" y2="73.66" width="0.1524" layer="91"/>
-<wire x1="-96.52" y1="73.66" x2="-99.06" y2="73.66" width="0.1524" layer="91"/>
-<wire x1="-96.52" y1="78.74" x2="-96.52" y2="73.66" width="0.1524" layer="91"/>
-<junction x="-96.52" y="73.66"/>
-<label x="-91.44" y="81.28" size="1.778" layer="95"/>
+<wire x1="-91.44" y1="73.66" x2="-93.98" y2="73.66" width="0.1524" layer="91"/>
+<wire x1="-93.98" y1="73.66" x2="-99.06" y2="73.66" width="0.1524" layer="91"/>
+<wire x1="-93.98" y1="78.74" x2="-93.98" y2="73.66" width="0.1524" layer="91"/>
+<junction x="-93.98" y="73.66"/>
+<label x="-88.9" y="83.82" size="1.778" layer="95"/>
 <pinref part="C3" gate="G$1" pin="2"/>
 <pinref part="IC2" gate="1" pin="PC6(/RESET/PCINT14)"/>
@@
 </segment>
 <segment>
-<wire x1="-96.52" y1="88.9" x2="-96.52" y2="91.44" width="0.1524" layer="91"/>
+<wire x1="-93.98" y1="88.9" x2="-93.98" y2="91.44" width="0.1524" layer="91"/>
 <pinref part="R1" gate="G$1" pin="2"/>
 <pinref part="+3V3" gate="G$1" pin="+3V3"/>
@@
 </segment>
 <segment>
-<wire x1="-106.68" y1="81.28" x2="-124.46" y2="81.28" width="0.1524" layer="91"/>
-<pinref part="JP7" gate="G$1" pin="4"/>
-<pinref part="+3V10" gate="G$1" pin="+3V3"/>
-</segment>
-<segment>
 <pinref part="LED1" gate="G$1" pin="A"/>
 <pinref part="+3V1" gate="G$1" pin="+3V3"/>
@@
 </segment>
 </net>
-<net name="COIN" class="0">
+<net name="EXT_VSUPPLY" class="0">
 <segment>
 <wire x1="114.3" y1="109.22" x2="121.92" y2="109.22" width="0.1524" layer="91"/>
-<pinref part="G2" gate="G$1" pin="+"/>
 <pinref part="SW_PWR" gate="BEF1" pin="S"/>
 </segment>
-</net>
-<net name="EXTPWR" class="0">
+<segment>
+<wire x1="-114.3" y1="81.28" x2="-124.46" y2="81.28" width="0.1524" layer="91"/>
+<pinref part="JP7" gate="G$1" pin="4"/>
+<label x="-114.3" y="81.28" size="1.778" layer="95"/>
+</segment>
+</net>
+<net name="BATT" class="0">
 <segment>
 <wire x1="101.6" y1="104.14" x2="121.92" y2="104.14" width="0.1524" layer="91"/>
